File: stage-sensor/stage-sensor-board.kicad_pcb (KiCad board)
At the start: 2 copper layers, 19.4 x 19.4 mm, 11 parts, among them J1 STEMMA QT, U1 ICM 42605, U3 SHT45

Commit message: Stage sensor board V0.1.1
Switched out the vertical stemma QT for horizontal one. Funciontally equivalent to V0.1.1 WIll send this one over for production.
Parts:
- J1: footprint Connector_JST:JST_SH_BM04B-SRSS-TB_1x04-1MP_P1.00mm_Vertical -> Connector_JST:JST_SH_SM04B-SRSS-TB_1x04-1MP_P1.00mm_Horizontal
- moved J1 1.91 mm to (129.6, 99.9), turned to 180 degrees
Routing:
- net /SDA: track 51.8 -> 55.3 mm
- net GND: track 12.6 -> 15.7 mm, vias 6 -> 8
- net /SCL: track 53.0 -> 51.4 mm
Other:
- board text added: "JST SH"
- board text added: "Sample Chuck Sensor PCB V0.1.1"
- board text added: "UV Sensor OPT3002"
- board text removed: "JST SH 1mm"
- board text removed: "Sample Chuck Sensor PCB V0.1.0"
- board text removed: "UV Sensor"
